Commit message: modified the configuration

File: interbotix_descriptions/urdf/vx300s.urdf.xacro (robot description, xacro)
@@ -116,5 +116,5 @@
     <axis xyz="0 1 0"/>
     <limit effort="100" lower="${radians(-92)}" upper="${radians(101)}" velocity="${pi}"/>
-    <origin rpy="${pi} 0 0" xyz="0.05955 0 0.3"/>
+    <origin rpy="${pi} 0 0" xyz="0.05955 0 0.18"/>
     <parent link="$(arg robot_name)/upper_arm_link"/>
     <child link="$(arg robot_name)/upper_forearm_link"/>
@@ -152,5 +152,5 @@
     <axis xyz="1 0 0"/>
     <limit effort="100" lower="${radians(-180)}" upper="${radians(180)}" velocity="${pi}"/>
-    <origin rpy="0 0 0" xyz="0.2 0 0"/>
+    <origin rpy="0 0 0" xyz="0.15 0 0"/>
     <parent link="$(arg robot_name)/upper_forearm_link"/>
     <child link="$(arg robot_name)/lower_forearm_link"/>
